Commit message: Naro de dos piezas completo

File: naro_description/urdf/naro_geometric.urdf (robot description, URDF)
Before this commit: robot naro, 8 links, 7 joints
Links:
- removed link NaroBody_3_link
- removed link Naro_caudal_fin_link
- removed link Naro_dorsal_fin_down_link
- removed link Naro_dorsal_fin_up_link
- removed link Naro_pectoral_fin_left_link
- removed link Naro_pectoral_fin_right_link
- added link dummy_link
Joints:
- removed joint NaroBody_1_Naro_dorsal_fin_down_joint
- removed joint NaroBody_1_Naro_dorsal_fin_up_joint
- removed joint NaroBody_1_Naro_pectoral_fin_left_joint
- removed joint NaroBody_1_Naro_pectoral_fin_right_joint
- removed joint NaroBody_2_NaroBody_3_joint
- removed joint NaroBody_3_Naro_caudal_fin_joint
- added joint dummy_joint: type fixed, parent dummy_link, child base_link

Commit message: completa modelo geometrico de naro

File: naro_description/urdf/naro_geometric.urdf (robot description, URDF)
Before this commit: robot naro, 3 links, 2 joints
Links:
- added link NaroBody_3_link, mass 0.2; collision cylinder length=0.05357 radius=0.028605; visual cylinder length=0.05357 radius=0.028605
- added link Naro_caudal_fin_link, mass 0.2; collision cylinder length=0.006 radius=0.07; visual cylinder length=0.006 radius=0.07
- added link Naro_dorsal_fin_down_link, mass 0.05; collision box size=0.006 0.0147 0.05978; visual box size=0.0147 0.006 0.05978
- added link Naro_dorsal_fin_up_link, mass 0.05; collision box size=0.006 0.0147 0.05978; visual box size=0.0147 0.006 0.05978
- added link Naro_pectoral_fin_left_link, mass 0.05; collision box size=0.006 0.0147 0.05978; visual box size=0.006 0.0147 0.05978
- added link Naro_pectoral_fin_right_link, mass 0.1; collision box size=0.006 0.0147 0.05978; visual box size=0.006 0.0147 0.05978
Joints:
- added joint NaroBody_1_Naro_dorsal_fin_down_joint: type fixed, parent NaroBody_2_link, child Naro_dorsal_fin_down_link, origin xyz=-0.035795 0 0.0362 rpy=0 1.5707963267948966 0
- added joint NaroBody_1_Naro_dorsal_fin_up_joint: type fixed, parent NaroBody_2_link, child Naro_dorsal_fin_up_link, origin xyz=0.035795 0 0.0362 rpy=0 1.5707963267948966 0
- added joint NaroBody_1_Naro_pectoral_fin_left_joint: type revolute, parent base_link, child Naro_pectoral_fin_left_link, origin xyz=-0.04275 0.05489 0.04478 rpy=1.5707963267948966 0 0, axis 0 0 1, limit lower=-0.2 upper=0.2 effort=0.1 velocity=0.5
- added joint NaroBody_1_Naro_pectoral_fin_right_joint: type revolute, parent base_link, child Naro_pectoral_fin_right_link, origin xyz=-0.04275 -0.05489 0.04478 rpy=1.5707963267948966 0 0, axis 0 0 1, limit lower=-0.2 upper=0.2 effort=0.1 velocity=0.5
- added joint NaroBody_2_NaroBody_3_joint: type revolute, parent NaroBody_2_link, child NaroBody_3_link, origin xyz=0 0 0.0874 rpy=0 0 0, axis 1 0 0, limit lower=-0.2 upper=0.2 effort=5.0 velocity=1.0
- added joint NaroBody_3_Naro_caudal_fin_joint: type revolute, parent NaroBody_3_link, child Naro_caudal_fin_link, origin xyz=0 0 0.05357 rpy=1.5707963267948966 0 0, axis 1 0 0, limit lower=-0.2 upper=0.2 effort=5.0 velocity=1.0
