Commit message: Agrega un sensor laser a m2wr

File: m2wr_description/urdf/gazebo.xacro (robot description, xacro)
@@ -26,4 +26,35 @@
   </plugin>
 </gazebo>
+<gazebo reference="sensor_laser">
+  <sensor type="ray" name="head_hokuyo_sensor">
+    <pose>0 0 0 0 0 0</pose>
+    <visualize>false</visualize>
+    <update_rate>20</update_rate>
+    <ray>
+      <scan>
+        <horizontal>
+          <samples>720</samples>
+          <resolution>1</resolution>
+          <min_angle>-1.570796</min_angle>
+          <max_angle>1.570796</max_angle>
+        </horizontal>
+      </scan>
+      <range>
+        <min>0.10</min>
+        <max>10.0</max>
+        <resolution>0.01</resolution>
+      </range>
+      <noise>
+        <type>gaussian</type>
+        <mean>0.0</mean>
+        <stddev>0.01</stddev>
+      </noise>
+    </ray>
+    <plugin name="gazebo_ros_head_hokuyo_controller" filename="libgazebo_ros_laser.so">
+      <topicName>/m2wr/laser/scan</topicName>
+      <frameName>sensor_laser</frameName>
+    </plugin>
+  </sensor>
+</gazebo>
 <gazebo reference="link_chassis">
   <material>Gazebo/Orange</material>

File: m2wr_description/urdf/m2wr.xacro (robot description, xacro)
@@ -48,4 +48,29 @@
   </visual>
 </link>
+<link name="sensor_laser">
+  <inertial>
+    <origin xyz="0 0 0" rpy="0 0 0" />
+    <mass value="1" />
+    <xacro:cylinder_inertia mass="1" r="0.05" l="0.1" />
+  </inertial>
+  <visual>
+    <origin xyz="0 0 0" rpy="0 0 0" />
+    <geometry>
+      <cylinder radius="0.05" length="0.1"/>
+    </geometry>
+    <material name="white" />
+  </visual>
+  <collision>
+    <origin xyz="0 0 0" rpy="0 0 0"/>
+    <geometry>
+      <cylinder radius="0.05" length="0.1"/>
+    </geometry>
+  </collision>
+</link>
+<joint name="joint_sensor_laser" type="fixed">
+  <origin xyz="0.15 0 0.05" rpy="0 0 0"/>
+  <parent link="link_chassis"/>
+  <child link="sensor_laser"/>
+</joint>
 <xacro:link_wheel position="right"/>
 <xacro:joint_wheel position="right" y="0.15"/>

File: m2wr_description/urdf/macro.xacro (robot description, xacro)
@@ -32,3 +32,8 @@
 </joint>
 </xacro:macro>
+<xacro:macro name="cylinder_inertia" params="mass r l">
+  <inertia ixx="${mass*(3*r*r+l*l)/12}" ixy = "0" ixz = "0"
+           iyy="${mass*(3*r*r+l*l)/12}" iyz = "0"
+           izz="${mass*(r*r)/2}" />
+</xacro:macro>
 </robot>

Commit message: Probando el uso de plugins para Gazebo

File: m2wr_description/urdf/gazebo.xacro (robot description, xacro)
@@ -58,8 +58,12 @@
 </gazebo>
 <gazebo reference="link_chassis">
-  <material>Gazebo/Orange</material>
-</gazebo>
-<gazebo reference="caster_front_visual">
-  <material>Gazebo/Orange</material>
+  <visual name="caster_front_visual">
+    <material>
+      <script>
+        <uri>file://media/materials/scripts/gazebo.material</uri>
+        <name>Gazebo/Orange</name>
+      </script>
+    </material>
+  </visual>
 </gazebo>
 <gazebo reference="link_left_wheel">
